Commit message: Add sensor

File: ch_iii_working_with_ros_for_3d_modeling/src/rrbot_description/urdf/rrbot.urdf (robot description, URDF)
Before this commit: robot rrbot, 3 links, 2 joints
Links:
- added link camera_link, mass 1e-5; collision box size=0.05 0.05 0.05; visual box size=0.05 0.05 0.05
- added link hokuyo_link, mass 1e-5; collision box size=0.1 0.1 0.1; visual mesh filename=package://rrbot_description/meshes/hokuyo.dae
- added link link3, mass 1; collision box size=0.1 0.1 1; visual box size=0.1 0.1 1
Joints:
- added joint camera_joint: type fixed, parent link3, child camera_link, origin xyz=0.05 0 0.9 rpy=0 0 0, axis 0 1 0
- added joint hokuyo_joint: type fixed, parent link3, child hokuyo_link, origin xyz=0.0 0.0 0.975 rpy=0.0 0.0 0.0, axis 0 1 0
- added joint joint2: type revolute, parent link2, child link3, origin xyz=0 0.1 0.9 rpy=0 0 0, axis 0 1 0, limit lower=-3.141592653589793 upper=3.141592653589793 effort=300.0 velocity=10.0
- joint fixed: origin (none) -> xyz=0.0 0.0 0.0 rpy=0.0 0.0 0.0
- joint joint1: limit (none) -> lower=-3.141592653589793 upper=3.141592653589793 effort=300.0 velocity=10.0; type continuous -> revolute

File: ch_iii_working_with_ros_for_3d_modeling/src/rrbot_description/urdf/rrbot.xacro (robot description, xacro)
@@ -123,4 +123,61 @@
     </inertial>
   </link>
+  <!-- hokuyo laser joint -->
+  <joint name="hokuyo_joint" type="fixed">
+    <axis xyz="0 1 0"/>
+    <origin xyz="0.0 0.0 ${height3 - axel_offset/2}" rpy="0.0 0.0 0.0"/>
+    <parent link="link3"/>
+    <child link="hokuyo_link"/>
+  </joint>
+  <!-- hokuyo laser link -->
+  <link name="hokuyo_link">
+    <visual>
+      <origin xyz="0 0 0" rpy="0 0 0"/>
+      <geometry>
+        <mesh filename="package://rrbot_description/meshes/hokuyo.dae"/>
+      </geometry>
+    </visual>
+    <collision>
+      <origin xyz="0 0 0" rpy="0 0 0"/>
+      <geometry>
+        <box size="0.1 0.1 0.1"/>
+      </geometry>
+    </collision>
+    <inertial>
+      <mass value="1e-5" />
+      <origin xyz="0 0 0" rpy="0 0 0"/>
+      <inertia  ixx="1e-6" ixy="0" ixz="0"
+                iyy="1e-6" iyz="0"
+                izz="1e-6" />
+    </inertial>
+  </link>
+  <!-- Camera joint -->
+  <joint name="camera_joint" type="fixed">
+    <axis xyz="0 1 0" />
+    <origin xyz="${camera_link} 0 ${height3 - axel_offset*2}" rpy="0 0 0"/>
+    <parent link="link3"/>
+    <child link="camera_link"/>
+  </joint>
+  <!-- Camera link -->
+  <link name="camera_link">
+    <collision>
+      <origin xyz="0 0 0" rpy="0 0 0"/>
+      <geometry>
+    <box size="${camera_link} ${camera_link} ${camera_link}"/>
+      </geometry>
+    </collision>
+    <visual>
+      <origin xyz="0 0 0" rpy="0 0 0"/>
+      <geometry>
+    <box size="${camera_link} ${camera_link} ${camera_link}"/>
+      </geometry>
+      <material name="red"/>
+    </visual>
+    <inertial>
+      <mass value="1e-5" />
+      <origin xyz="0 0 0" rpy="0 0 0"/>
+      <inertia ixx="1e-6" ixy="0" ixz="0" iyy="1e-6" iyz="0" izz="1e-6" />
+    </inertial>
+  </link>
   <!-- TRANSMISSIONS -->
   <xacro:transmission_block trans="trans1" joint="joint1" motor="motor1"/>
