Commit message: Add robot simulation with gazebo

File: ch04/src/seven_dof_robot_description/urdf/materials.xacro (robot description, xacro)
@@ -11,3 +11,6 @@
     <color rgba="1.0 1.0 1.0 1.0"/>
   </material>
+  <material name="Blue">
+    <color rgba="0.0 0.0 1.0 1.0"/>
+  </material>
 </robot>

File: ch04/src/seven_dof_robot_description/urdf/sensors/xtion_pro_live.xacro (robot description, xacro)
@@ -12,4 +12,7 @@
   </xacro:macro>
   <xacro:macro name="xtion_pro_live" params="name parent *origin *optical_origin">
+  <material name="DarkGrey">
+    <color rgba="${88/255} ${88/255} ${88/255} 1.0"/>
+  </material>
     <!-- frames in the center of the camera -->
     <joint name="${name}_joint" type="fixed">

File: ch04/src/seven_dof_robot_description/urdf/seven_dof_arm_rgbd.xacro (robot description, xacro)
@@ -57,14 +57,14 @@
   <!-- xacro:macro for transmission block -->
   <xacro:macro name="transmission_block" params="trans_name joint_name motor_name">
-    <transmision name="${trans_name}">
-      <type>transmission_interface/SimpleTransmission</type>
-      <joint name="${joint_name}">
-        <hardwareInterface>hardware_interface/PositionJointInterface</hardwareInterface>
-      </joint>
-      <actuator name="${motor_name}">
-        <hardwareInterface>hardware_interface/PositionJointInterface</hardwareInterface>
-        <mechanicalReduction>1</mechanicalReduction>
-      </actuator>
-    </transmision>
+    <transmission name="${trans_name}">
+    <type>transmission_interface/SimpleTransmission</type>
+    <joint name="${joint_name}">
+      <hardwareInterface>hardware_interface/PositionJointInterface</hardwareInterface>
+    </joint>
+    <actuator name="${motor_name}">
+      <hardwareInterface>hardware_interface/PositionJointInterface</hardwareInterface>
+      <mechanicalReduction>1</mechanicalReduction>
+    </actuator>
+  </transmission>
   </xacro:macro>
     <!-- LINKS AND JOINTS -->
@@ -107,5 +107,5 @@
         <box size="0.1 0.1 0.1"/>
       </geometry>
-      <material name="Gray"/>
+      <material name="White"/>
     </visual>
     <collision>
@@ -133,4 +133,5 @@
         <cylinder radius="${shoulder_pan_width}" length="${shoulder_pan_len}"/>
       </geometry>
+      <material name="Red"/>
     </visual>
     <collision>
@@ -156,5 +157,5 @@
         <box size="${shoulder_pitch_len} ${shoulder_pitch_width} ${shoulder_pitch_height}"/>
       </geometry>
-      <material name="Gray"/>
+      <material name="White"/>
     </visual>
     <collision>
@@ -258,5 +259,5 @@
         <box size="${wrist_pitch_len} ${wrist_pitch_width} ${wrist_pitch_height}"/>
       </geometry>
-      <material name="Gray"/>
+      <material name="White"/>
     </visual>
     <collision>
@@ -310,5 +311,5 @@
         <box size="${left_gripper_len} ${left_gripper_width} ${left_gripper_height}"/>
       </geometry>
-      <material name="Gray"/>
+      <material name="White"/>
     </visual>
     <collision>
@@ -341,5 +342,5 @@
         <box size="${right_gripper_len} ${right_gripper_width} ${right_gripper_height}"/>
       </geometry>
-      <material name="Gray"/>
+      <material name="White"/>
     </visual>
     <collision>
@@ -363,5 +364,5 @@
         <box size="0.01 0.01 0.01"/>
       </geometry>
-      <material name="White"/>
+      <material name="Blue"/>
     </visual>
     <inertial>
@@ -383,4 +384,14 @@
   </xacro:xtion_pro_live>
   <!-- TRANSMISSIONS -->
+  <!-- <transmission name="tran1">
+    <type>transmission_interface/SimpleTransmission</type>
+    <joint name="shoulder_pan_joint">
+      <hardwareInterface>hardware_interface/PositionJointInterface</hardwareInterface>
+    </joint>
+    <actuator name="motor1">
+      <hardwareInterface>hardware_interface/PositionJointInterface</hardwareInterface>
+      <mechanicalReduction>1</mechanicalReduction>
+    </actuator>
+  </transmission> -->
   <xacro:transmission_block trans_name="trans1" joint_name="shoulder_pan_joint" motor_name="motor1"/>
   <xacro:transmission_block trans_name="trans2" joint_name="shoulder_pitch_joint" motor_name="motor2"/>
@@ -390,5 +401,5 @@
   <xacro:transmission_block trans_name="trans6" joint_name="wrist_pitch_joint" motor_name="motor6"/>
   <xacro:transmission_block trans_name="trans7" joint_name="gripper_roll_joint" motor_name="motor7"/>
-  <xacro:transmission_block trans_name="trans7" joint_name="finger_joint1" motor_name="motor7"/>
-  <xacro:transmission_block trans_name="trans7" joint_name="finger_joint2" motor_name="motor7"/>
+  <xacro:transmission_block trans_name="trans8" joint_name="finger_joint1" motor_name="motor8"/>
+  <xacro:transmission_block trans_name="trans9" joint_name="finger_joint2" motor_name="motor9"/>
 </robot>
